Commit message: sp

File: semester_M1_2/src/my_urdf/urdf/robot.xacro (robot description, xacro)
@@ -1,9 +1,9 @@
-<robot xmlns:xacro="http://www.ros.org/wiki/xacro" name="my_robot">
+<robot xmlns:xacro="http://www.ros.org/wiki/xacro" name="robot">
     <xacro:property name="wheel_thickness" value="0.06" />
-    <xacro:property name="wheel_radius" value="0.063" />
+    <xacro:property name="wheel_radius" value="0.1" />
     <xacro:property name="roller_radius" value="0.1075" />
-    <xacro:property name="body_length" value="0.380" />
-    <xacro:property name="body_width" value="0.120" />
-    <xacro:property name="body_height" value="0.072" />
+    <xacro:property name="body_length" value="0.497" />
+    <xacro:property name="body_width" value="0.274" />
+    <xacro:property name="body_height" value="0.191" />
     <xacro:property name="mass" value="3.3" />
     <xacro:property name="wheel_mass" value="1e-5" />
@@ -11,18 +11,7 @@
     <!-- Import all Gazebo-customization elements, including Gazebo colors -->
     <xacro:include filename="$(find my_urdf)/urdf/robot.gazebo" />
-    <material name="blue">
-        <color rgba="0 0 0.8 1"/>
-    </material>
-    <material name="black">
-        <color rgba="0 0 0 1"/>
-    </material>
-    <material name="white">
-        <color rgba="1 1 1 1"/>
-    </material>
-    <material name="gray">
-        <color rgba="0.7 0.7 0.7 1"/>
-    </material>
-    <link name="world"/>
-    <joint name="fixed" type="fixed">
+    <xacro:include filename="utils.xacro" />
+    <link name="world" />
+    <joint name="fixed=" type="fixed">
         <parent link="world"/>
         <child link="base_link"/>
@@ -30,22 +19,22 @@
     <link name="base_link">
         <visual>
-            <origin xyz="0.0 0.0 ${body_height/2}"/>
-            <geometry>
-                <mesh filename="package://my_urdf/meshes/chassis.dae" scale="${body_length*2.3} ${body_width*3.6} ${body_height*5.71}"/>
-            </geometry>
-        </visual>
-        <collision>
-            <origin xyz="0.0 0.0 ${body_height/2}"/>
-            <geometry>
-                <box size="${body_length} ${body_width} ${body_height}"/>
-            </geometry>
-        </collision>
-        <inertial>
-            <!-- <origin xyz="0.0 0.0 ${body_height/2+0.09}"/> -->
-            <mass value="3.3" /> <!-- mass in kg -->
-            <inertia ixx="0.005386" ixy="0.000000" ixz="0.00000"
-                                        iyy="0.041136" iyz="0.00000"
-                                                       izz="0.04367"/>
-            </inertial>
+            <geometry>
+                <mesh filename="package://my_urdf/meshes/chassis.dae"/>
+            </geometry>
+        </visual>
+        <collision>
+            <geometry>
+                <mesh filename="package://my_urdf/meshes/chassis.dae"/>
+            </geometry>
+        </collision>
+        <xacro:inertial_box mass="0.5" x="${body_length}" y="${body_width}" z="${body_height}">
+            <origin xyz="0 0 0" rpy="0 0 0"/>
+        </xacro:inertial_box>
+        <!-- <inertial>
+            <mass value="3" />
+            <inertia ixx="0.20378242" ixy="0.000000" ixz="0.00000"
+                     iyy="0.0619377" iyz="0.00000"
+                     izz="0.03009682"/>
+        </inertial> -->
     </link>
     <xacro:macro name="wheel" params="prefix color radius thickness reflect">
@@ -53,7 +42,7 @@
             <parent link="base_link"/>
             <child link="${prefix}_wheel"/>
-            <origin xyz="${-body_length/4} ${reflect*(body_width/2+thickness/2)} 0"/>
+            <origin xyz="${-body_length/4} ${reflect*(body_width/2+thickness/2)} ${-radius}" rpy="0 0 0"/>
             <axis xyz = "0 1 0" />
-            <dynamics damping ="0.002" />
+            <dynamics damping="0.02" />
         </joint>
         <link name="${prefix}_wheel">
@@ -61,5 +50,6 @@
                 <origin rpy="${pi/2} 0.0 0.0"/>
                 <geometry>
-                    <cylinder radius="${radius}" length="${thickness}"/>
+                    <box size="${radius*2} ${radius} ${thickness}"/>
+                    <!-- <cylinder radius="${radius}" length="${thickness}"/> -->
                 </geometry>
                 <material name="${color}"/>
@@ -68,21 +58,26 @@
                 <origin xyz="0 ${thickness/2 + 0.002} 0" rpy="${pi/2} 0 0"/>
                 <geometry>
-                    <cylinder radius="${radius}" length="${thickness}"/>
+                    <box size="${radius*2} ${radius} ${thickness}"/>
+                    <!-- <cylinder radius="${radius}" length="${thickness}"/> -->
                 </geometry>
             </collision>
-            <inertial>
+            <xacro:inertial_cylinder mass="1.0" length="${wheel_thickness}" radius="${wheel_radius}">
+                <origin xyz="0 ${wheel_thickness/2} 0" rpy="${pi/2} 0 0"/>
+            </xacro:inertial_cylinder>
+            <!-- <inertial>
                 <mass value="0.150"/>
                 <inertia ixx="0.00019384" ixy="0.00000000" ixz="00000000"
                                           iyy="0.00019384" iyz="00000000"
                                                            izz="0.004725"/>
-            </inertial>
+            </inertial> -->
         </link>
     </xacro:macro>
     <xacro:wheel prefix="left" color="black" radius="${wheel_radius}" thickness="${wheel_thickness}" reflect="1"/>
     <xacro:wheel prefix="right" color="blue" radius="${wheel_radius}" thickness="${wheel_thickness}" reflect="-1"/>
+    <!-- Roller  -->
     <joint name="roller_wheel_horizontal_to_base" type="continuous">
         <parent link="base_link"/>
         <child link="roller_wheel_horizontal"/>
-        <origin xyz="${body_length/2 - wheel_radius / 2} 0.0 -${wheel_radius / 2}"/>
+        <origin xyz="${body_length/2 - wheel_radius / 2} 0.0 ${-body_height/2-wheel_radius/2}"/>
 		<axis xyz = "0 0 1" />
 		<dynamics damping ="0.002" />
@@ -102,10 +97,13 @@
             </geometry>
         </collision>
-        <inertial>
+        <xacro:inertial_sphere mass="1" radius="${wheel_radius}">
+            <origin rpy="${pi/2} 0.0 0.0"/>
+        </xacro:inertial_sphere>
+        <!-- <inertial>
             <mass value="0.150"/>
             <inertia ixx="0.00019384" ixy="0.00000000" ixz="00000000"
                                         iyy="0.00019384" iyz="00000000"
                                                         izz="0.004725"/>
-        </inertial>
+        </inertial> -->
     </link>
     <joint name="roller_wheel_vertical_to_base" type="continuous">
@@ -129,5 +127,8 @@
             </geometry>
         </collision>
-        <inertial>
+        <xacro:inertial_sphere mass="1" radius="${wheel_radius}">
+            <origin rpy="${pi/2} 0.0 0.0"/>
+        </xacro:inertial_sphere>
+        <!-- <inertial>
             <origin rpy="${pi/2} 0.0 0.0"/>
             <mass value="0.15" />
@@ -135,22 +136,10 @@
                     iyy="0.0001" iyz="0"
                     izz="0.0001" />
-        </inertial>
-    </link>
-    <!-- <link name="chassis">
-        <visual>
-            <origin xyz="0 0 0.3"/>
-            <geometry>
-                <mesh filename="package://my_urdf/meshes/chassis.dae"/>
-            </geometry>
-        </visual>
-    </link>
-    <joint name="chassis_joint" type="fixed">
-        <parent link="base_link"/>
-        <child link="chassis"/>
-    </joint> -->
+        </inertial> -->
+    </link>
     <!-- Hokuyo Laser -->
     <joint name="hokuyo_joint" type="fixed">
         <axis xyz="0 1 0" />
-        <origin xyz="0 0 0.2" rpy="0 0 0"/>
+        <origin xyz="0 0 ${body_height/2}" rpy="0 0 0"/>
         <parent link="base_link"/>
         <child link="hokuyo_link"/>
@@ -175,3 +164,70 @@
         </inertial>
     </link>
+    <joint name="bamper_joint" type="fixed">
+        <axis xyz="0 1 0" />
+        <origin xyz="0 0 ${body_height/2}" rpy="0 0 0"/>
+        <parent link="base_link"/>
+        <child link="bumper_link"/>
+    </joint>
+    <link name="bumper_link">
+        <collision>
+            <origin xyz="0 0 -0.01" rpy="0 0 0"/>
+            <geometry>
+                <box size="0.3 0.075 0.025"/>
+            </geometry>
+        </collision>
+        <visual>
+            <origin xyz="0 0 -0.01" rpy="0 0 0"/>
+            <geometry>
+                <box size="0.3 0.075 0.025"/>
+            </geometry>
+            <material name="red"/>
+        </visual>
+        <inertial>
+            <mass value="1e-5" />
+            <origin xyz="0 0 -0.01" rpy="0 0 0"/>
+            <inertia ixx="1e-6" ixy="0" ixz="0" iyy="1e-6" iyz="0" izz="1e-6" />
+        </inertial>
+    </link>
+    <!-- transmissions -->
+    <transmission name="roller_wheel_horizontal_tran">
+        <type>transmission_interface/SimpleTransmission</type>
+        <joint name="roller_wheel_horizontal_to_base">
+        <hardwareInterface>hardware_interface/EffortJointInterface</hardwareInterface>
+        </joint>
+        <actuator name="roller_wheel_horizontal_motor">
+        <hardwareInterface>hardware_interface/EffortJointInterface</hardwareInterface>
+        <mechanicalReduction>1</mechanicalReduction>
+        </actuator>
+    </transmission>
+    <transmission name="roller_wheel_vertical_tran">
+        <type>transmission_interface/SimpleTransmission</type>
+        <joint name="roller_wheel_vertical_to_base">
+        <hardwareInterface>hardware_interface/EffortJointInterface</hardwareInterface>
+        </joint>
+        <actuator name="roller_wheel_vertical_motor">
+        <hardwareInterface>hardware_interface/EffortJointInterface</hardwareInterface>
+        <mechanicalReduction>1</mechanicalReduction>
+        </actuator>
+    </transmission>
+    <transmission name="left_wheel_trans">
+        <type>transmission_interface/SimpleTransmission</type>
+        <joint name="joint_left_wheel_to_base">
+            <hardwareInterface>hardware_interface/EffortJointInterface</hardwareInterface>
+        </joint>
+        <actuator name="left_wheel_motor">
+            <mechanicalReduction>1.0</mechanicalReduction>
+            <hardwareInterface>hardware_interface/EffortJointInterface</hardwareInterface>
+        </actuator>
+    </transmission>
+    <transmission name="right_wheel_trans">
+        <type>transmission_interface/SimpleTransmission</type>
+        <joint name="joint_right_wheel_to_base">
+            <hardwareInterface>hardware_interface/EffortJointInterface</hardwareInterface>
+        </joint>
+        <actuator name="right_wheel_motor">
+            <mechanicalReduction>1.0</mechanicalReduction>
+            <hardwareInterface>hardware_interface/EffortJointInterface</hardwareInterface>
+        </actuator>
+    </transmission>
 </robot>

Commit message: sp

File: semester_M1_2/src/my_urdf/urdf/robot.xacro (robot description, xacro)
@@ -12,9 +12,9 @@
     <xacro:include filename="$(find my_urdf)/urdf/robot.gazebo" />
     <xacro:include filename="utils.xacro" />
-    <link name="world" />
+    <!-- <link name="world" />
     <joint name="fixed=" type="fixed">
         <parent link="world"/>
         <child link="base_link"/>
-    </joint>
+    </joint> -->
     <link name="base_link">
         <visual>
